File: led_driver_test_board/led_driver_test_board.kicad_pcb (KiCad board)
At the start: 2 copper layers, 39 x 52.8 mm, 124 parts, among them P1 CONN_01X06_M50-3530642, P2 CONN_01X06_M50-3530642, P3 CONN_01X06_M50-3530642, P4 CONN_01X06_M50-3530642, P5 CONN_01X06_M50-3530642, Q1 Q_NMOS_SSM3K09FULF, Q2 Q_NMOS_SSM3K09FULF, Q3 Q_NMOS_SSM3K09FULF, Q4 Q_NMOS_SSM3K09FULF, Q5 Q_NMOS_SSM3K09FULF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

Commit message: Updated title block to current revision 1.1
Other:
- board text added: "1.1"
- board text added: "12/27/2017"
- board text added: "ZERO GECKO BREAKOUT FOR LED DRIVER TESTING"
- board text added: "led_driver_test_board.kicad_pcb"
Changed lines of the file:
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@@
 (kicad_pcb (version 4) (host pcbnew 4.0.2+dfsg1-stable)
   (general
-    (links 0)
+    (links 219)
     (no_connects 0)
     (area 91.275212 44.237286 147.167477 108.217476)
     (thickness 1.6)
-    (drawings 39)
+    (drawings 43)
     (tracks 1070)
     (zones 0)
@@
     (46 B.CrtYd user hide)
     (47 F.CrtYd user hide)
-    (48 B.Fab user hide)
+    (48 B.Fab user)
     (49 F.Fab user hide)
   )
@@
       (xy -3.888879 5.690484)) (layer B.SilkS) (width 0.01))
   )
+  (gr_text 1.1 (at 270.3 193.1) (layer Dwgs.User)
+    (effects (font (size 1.5 1.5) (thickness 0.3)))
+  )
+  (gr_text 12/27/2017 (at 213.5 193.1) (layer Dwgs.User)
+    (effects (font (size 1.5 1.5) (thickness 0.3)))
+  )
+  (gr_text led_driver_test_board.kicad_pcb (at 201.1 185.9) (layer Dwgs.User)
+    (effects (font (size 1.5 1.5) (thickness 0.3)))
+  )
+  (gr_text "ZERO GECKO BREAKOUT FOR LED DRIVER TESTING" (at 214.7 189.5) (layer Dwgs.User)
+    (effects (font (size 1.5 1.5) (thickness 0.3)))
+  )
   (gr_text "LED BREAKOUT\n12_30_2017\nV1.1" (at 107.75 97.85 90) (layer F.SilkS)
